File: PCB PFC/PCB PFC.kicad_sch (KiCad schematic)
At the start: 48 parts, among them J4 External_Power, J5 JUMPER_BAT54S, SW2 SW_Push, U1 INA128, U3 TL082, U4 TL084, U5 TL082, U8 ESP32-C3_SUPERMINI_TH

Commit message: cambio de un valor de resistencia kicad
Parts:
- RfAD1: value 4.8k -> 10k
Changed lines of the file:
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@@
 			)
 		)
-		(property "Value" "4.8k"
+		(property "Value" "10k"
 			(at 220.98 96.52 90)
 			(effects

Commit message: comentarios
Other:
- note added: "en la placa 2, el CHP2 es de 10nf"
Changed lines of the file:
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@@
+		)
+	)
+	(text "en la placa 2, el CHP2 es de 10nf"
+		(exclude_from_sim no)
+		(at 157.48 16.764 0)
+		(effects
+			(font
+				(size 1.27 1.27)
+			)
 		)
 	)

Commit message: cambio R amp hw
Parts:
- RiAD1: value 1k -> 500
Changed lines of the file:
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@@
 			)
 		)
-		(property "Value" "1k"
+		(property "Value" "500"
 			(at 201.93 105.41 90)
 			(effects

Commit message: Actualización del esquemático
Parts:
- R10: value 16.2k -> 10k
- R9: value 1k -> 210
Changed lines of the file:
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@@
 			)
 		)
-		(property "Value" "1k"
+		(property "Value" "210"
 			(at 213.36 36.83 90)
 			(effects
@@
 			)
 		)
-		(property "Value" "16.2k"
+		(property "Value" "10k"
 			(at 226.06 52.578 90)
 			(effects
