File: PCB PFC/PCB PFC.kicad_sch (KiCad schematic)
At the start: 48 parts, among them J4 External_Power, J5 JUMPER_BAT54S, SW2 SW_Push, U1 INA128, U3 TL082, U4 TL084, U5 TL082, U8 ESP32-C3_SUPERMINI_TH

Commit message: KiCad: valores confirmados en banco (CHP1, CHP2, R8, RiAD1, INA122)
Cinco valores que estaban confirmados sin ambiguedad:

  CHP1    4.7n   -> 20n     confirmado por Luca
  CHP2    1.5n   -> 10n     confirmado por Luca
  R8      10k    -> 8.2k    anotado en la hoja de banco del 15/09
  RiAD1   500    -> 1k      nota de la hoja: "Cambio RiAD1 500 -> 1K"
  U1      INA128 -> INA122  el chip real; el BOM mandaba a comprar el equivocado

El lib_id de U1 sigue siendo Amplifier_Instrumentation:INA128. Mismo pinout
SOIC-8, asi que la placa y el footprint no cambian, pero el valor que se ve
en el esquematico y el que sale al BOM ahora dicen INA122, que es lo que
importa para no volver a comprar el chip equivocado.

RiAD1 explica que fue "ajustar la ganancia del Howland": el generador paso de
ganancia 20 (10k/500) a 10 (10k/1k). Con 20, U3A tendria que sacar ~6,4 Vpp
contra rieles de +-3,7 V, o sea estaba recortando.

Y cierra con el 8,06 k medido en circuito: con RfAD1=10k, RiAD1=1k y
rhpad1=500 el camino paralelo es 41,5k, y 10k || 41,5k = 8,058k. Exacto. O
sea RfAD1 NO cambio, sigue en 10k.

SIN TOCAR, esperando medicion con una pata levantada:
  R10    el archivo dice 16,2k y la hoja impresa dice 10k. De esto depende
         R9: con R10=10k, R9=2,2k; con R10=16,2k, R9=3,7k
  R9     la hoja tiene algo entre "22K" y "2,2K"
  CLP2   el archivo dice 270p, la atenuacion medida de U4C pide ~458p
  RfAD1  la hoja dice "8K" pero todo lo demas dice 10k

Ninguno de esos cuatro afecta K_CAL: la cadena se toma punta a punta.

El PCB sigue desincronizado del esquematico (nunca se corrio "Actualizar PCB
desde esquematico"). Esto no lo cambia.

Incluye tambien las ediciones de texto del cajetin que estaban sin commitear
(fecha 10/12/25 -> 4/9/26 y la nota "Correccion de comp").

Co-Authored-By: Claude Opus 5 <noreply@anthropic.com>
Claude-Session: https://claude.ai/code/session_01LfmR26CcbFRkuntFbsCN2c
Parts:
- CHP1: value 4.7n -> 20n
- CHP2: value 1.5n -> 10n
- R8: value 10k -> 8.2k
- RiAD1: value 500 -> 1k
- U1: value INA128 -> INA122
Other:
- note added: "4/9/26"
- note added: "Correccion de comp"
- note removed: "10/12/25"
- note removed: "Incorporo componentes SMD"
Changed lines of the file:
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@@
 		)
 	)
-	(text "10/12/25"
+	(text "4/9/26"
 		(exclude_from_sim no)
-		(at 198.628 189.738 0)
+		(at 217.17 193.548 0)
 		(effects
 			(font
@@
 		)
 	)
-	(text "Incorporo componentes SMD\n\n"
+	(text "Correccion de comp"
 		(exclude_from_sim no)
 		(at 224.79 170.18 0)
@@
 			)
 		)
-		(property "Value" "10k"
+		(property "Value" "8.2k"
 			(at 185.42 37.592 90)
 			(effects
@@
 			)
 		)
-		(property "Value" "INA128"
+		(property "Value" "INA122"
 			(at 42.418 61.722 0)
 			(effects
@@
 			)
 		)
-		(property "Value" "4.7n"
+		(property "Value" "20n"
 			(at 118.11 35.56 90)
 			(effects
@@
 			)
 		)
-		(property "Value" "500"
+		(property "Value" "1k"
 			(at 201.93 105.41 90)
 			(effects
@@
 			)
 		)
-		(property "Value" "1.5n"
+		(property "Value" "10n"
 			(at 152.4 35.56 90)
 			(effects
