File: PCB PFC/PCB PFC.kicad_sch (KiCad schematic)
At the start: 48 parts, among them J4 External_Power, J5 JUMPER_BAT54S, SW2 SW_Push, U1 INA122, U3 TL082, U4 TL084, U5 TL082, U8 ESP32-C3_SUPERMINI_TH

Commit message: comentario en kicad y resist
Parts:
- R9: value 210 -> 2,2k
Other:
- note added: "en alguna placa nueva es R9=1,1k"
Changed lines of the file:
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@@
 		)
 	)
+	(text "en alguna placa nueva es R9=1,1k\n"
+		(exclude_from_sim no)
+		(at 210.312 17.78 0)
+		(effects
+			(font
+				(size 1.27 1.27)
+			)
+		)
+	)
 	(text "16/9/26"
 		(exclude_from_sim no)
@@
 			)
 		)
-		(property "Value" "210"
+		(property "Value" "2,2k"
 			(at 213.36 36.83 90)
 			(effects
